Commit message: Fix model

File: 02_Impl/02_Source/Simulation/ROVER_1000_WATT_VARIANT.SLDASM/urdf/ROVER_1000_WATT_VARIANT.SLDASM.urdf (robot description, URDF)
Before this commit: robot ROVER_1000_WATT_VARIANT.SLDASM, 5 links, 4 joints
Links:
- added link base_footprint
- link base_link: mass 33.4459522433341 -> 35.6474447622668; geometry collision box size=0.823 0.5 0.575; visual mesh filename=package://ROVER_1000_WATT_VARIANT.SLDASM/meshes/base_link.S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
- link link_back_left: mass 7.01210916317506 -> 5.0741; geometry collision cylinder length=0.108 radius=0.1699; visual mesh filename=package://ROVER_1000_WATT_VARIANT.SLDASM/meshes/link_back_l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
- link link_back_right: mass 7.01210916337626 -> 5.0741; geometry collision cylinder length=0.108 radius=0.1699; visual mesh filename=package://ROVER_1000_WATT_VARIANT.SLDASM/meshes/link_back_r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
- link link_front_left: mass 7.01210916352614 -> 5.0741; geometry collision cylinder length=0.108 radius=0.1699; visual mesh filename=package://ROVER_1000_WATT_VARIANT.SLDASM/meshes/link_front_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
- link link_front_right: mass 7.01210916309939 -> 5.0741; geometry collision cylinder length=0.108 radius=0.1699; visual mesh filename=package://ROVER_1000_WATT_VARIANT.SLDASM/meshes/link_front_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
Joints:
- added joint base_footprint_joint: type fixed, parent base_footprint, child base_link, origin xyz=0 0 0.132487 rpy=0 0 0
- joint joint_back_left: origin xyz=-0.25123 0.31801 0.033 rpy=0 0 0 -> xyz=-0.25156 0.30851 0.037363 rpy=0 0 0
- joint joint_back_right: origin xyz=-0.25123 -0.31801 0.033 rpy=0 0 0 -> xyz=-0.25156 -0.30851 0.037363 rpy=0 0 0
- joint joint_front_left: origin xyz=0.25117 0.31801 0.033 rpy=0 0 0 -> xyz=0.2515 0.30851 0.037363 rpy=0 0 0
- joint joint_front_right: origin xyz=0.25117 -0.31801 0.033 rpy=0 0 0 -> xyz=0.2515 -0.30851 0.037363 rpy=0 0 0

Commit message: Update URDF

File: 02_Impl/02_Source/Simulation/ROVER_1000_WATT_VARIANT.SLDASM/urdf/ROVER_1000_WATT_VARIANT.SLDASM.urdf (robot description, URDF)
Before this commit: robot ROVER_1000_WATT_VARIANT.SLDASM, 6 links, 5 joints
Links:
- removed link base_footprint
- link base_link: mass 35.6474447622668 -> 37.2297696413548; geometry collision mesh filename=package://ROVER_1000_WATT_VARIANT.SLDASM/meshes/base_link.S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; visual mesh filename=package://ROVER_1000_WATT_VARIANT.SLDASM/meshes/base_link.S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
- link link_back_left: geometry collision mesh filename=package://ROVER_1000_WATT_VARIANT.SLDASM/meshes/link_back_l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; visual mesh filename=package://ROVER_1000_WATT_VARIANT.SLDASM/meshes/link_back_l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
- link link_back_right: geometry collision mesh filename=package://ROVER_1000_WATT_VARIANT.SLDASM/meshes/link_back_r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; visual mesh filename=package://ROVER_1000_WATT_VARIANT.SLDASM/meshes/link_back_r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
- link link_front_left: geometry collision mesh filename=package://ROVER_1000_WATT_VARIANT.SLDASM/meshes/link_front_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; visual mesh filename=package://ROVER_1000_WATT_VARIANT.SLDASM/meshes/link_front_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
- link link_front_right: geometry collision mesh filename=package://ROVER_1000_WATT_VARIANT.SLDASM/meshes/link_front_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; visual mesh filename=package://ROVER_1000_WATT_VARIANT.SLDASM/meshes/link_front_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
Joints:
- removed joint base_footprint_joint

Commit message: Update model

File: 02_Impl/02_Source/Simulation/ROVER_1000_WATT_VARIANT.SLDASM/urdf/ROVER_1000_WATT_VARIANT.SLDASM.urdf (robot description, URDF)
Before this commit: robot ROVER_1000_WATT_VARIANT.SLDASM, 5 links, 4 joints
Links:
- link base_link: mass 37.2297696413548 -> 37.356
